Commit message: Checkpoint before local-planner recovery-behavior rewrite
Command pipeline (goal_bridge, vlm_bridge, locations) and full-survey
course support; visibility-fan-filled local occupancy grid in
dwa_controller with obstacle inflation; DWA forward/reverse hysteresis,
debounce, and lane-check state machine in dwa.py; camera-pole/LIDAR
minRange fixes in the URDF/xacro/USD; AMCL particle-count and update
threshold tuning for the repetitive office layout.

Saving this as a checkpoint before replacing the reverse-hysteresis
approach in dwa.py with a bounded recovery-behavior pattern (stuck
detection + fixed-distance backup, rather than cost-margin tuning).

Co-Authored-By: Claude Sonnet 5 <noreply@anthropic.com>

File: jetracer.urdf (robot description, URDF)
Before this commit: robot jetracer, 12 links, 11 joints
Links:
- link camera: geometry collision cylinder length=0.006 radius=0.0075; visual cylinder length=0.006 radius=0.0075
- link camera_mount: geometry collision box size=0.01 0.01 0.20; visual box size=0.01 0.01 0.20
Joints:
- joint camera_joint: origin xyz=0 0 0.06 rpy=0 1.920 0 -> xyz=0 0 0.103 rpy=0 0 0

File: jetracer.xacro (robot description, xacro)
@@ -155,5 +155,5 @@
             <origin xyz="0.0 0.0 0.0" rpy="0.0 0.0 0.0"/>
             <geometry>
-                <box size="0.01 0.01 0.10"/>
+                <box size="0.01 0.01 0.20"/>
             </geometry>
             <material name="mount_red">
@@ -164,10 +164,10 @@
             <origin xyz="0.0 0.0 0.0" rpy="0.0 0.0 0.0"/>
             <geometry>
-                <box size="0.01 0.01 0.10"/>
+                <box size="0.01 0.01 0.20"/>
             </geometry>
         </collision>
     </link>
     <joint name="camera_joint" type="fixed">
-        <origin xyz="0 0 0.06" rpy="0 1.920 0"/>
+        <origin xyz="0 0 0.103" rpy="0 0 0"/>
         <parent link="camera_mount"/>
         <child link="camera"/>
@@ -182,5 +182,5 @@
             <origin xyz="0 0 0" rpy="0 0 0"/>
             <geometry>
-                <cylinder radius="0.0075" length="0.02"/>
+                <cylinder radius="0.0075" length="0.006"/>
             </geometry>
             <material name="camera_black">
@@ -191,5 +191,5 @@
             <origin xyz="0 0 0" rpy="0 0 0"/>
             <geometry>
-                <cylinder radius="0.0075" length="0.02"/>
+                <cylinder radius="0.0075" length="0.006"/>
             </geometry>
         </collision>
