Commit message: Add DWA local controller and navigation launch file, wire up A*/DWA stack
Adds primitives/utils/dwa/dwa_controller for Ackermann-adapted DWA local
control following the A* global plan, plus navigation_launch.py to run
both together. Also includes updated maps/slam config, lidar debug-draw
disabled in jetracer.usda, and .gitignore for colcon build artifacts.

File: jetracer.urdf (robot description, URDF)
Before this commit: robot jetracer, 12 links, 11 joints
Links:
- removed link base
- added link base_link, mass 1.0; collision box size=0.22 0.11 0.02; visual box size=0.22 0.11 0.02
Joints:
- joint board_joint: parent base -> base_link
- joint camera_joint: origin xyz=0 0 0.06 rpy=0 -0.349 0 -> xyz=0 0 0.06 rpy=0 1.920 0
- joint camera_mount_joint: parent base -> base_link
- joint front_left_base_holder: parent base -> base_link
- joint front_right_base_holder: parent base -> base_link
- joint head_joint: parent base -> base_link
- joint rear_left_wheel_joint: parent base -> base_link
- joint rear_right_wheel_joint: parent base -> base_link

File: jetracer.xacro (robot description, xacro)
@@ -5,5 +5,5 @@
     </material>
     <!-- Main Base -->
-    <link name="base">
+    <link name="base_link">
         <visual>
             <origin rpy="0 0 0" xyz="0 0 0"/>
@@ -31,5 +31,5 @@
             <axis xyz="0 0 1"/>
             <origin rpy="-1.57 0.0 0.0" xyz="${x} ${y} -0.01"/>
-            <parent link="base"/>
+            <parent link="base_link"/>
             <child link="${prefix}_wheel"/>
         </joint>
@@ -59,5 +59,5 @@
             <axis xyz="0 0 1"/>
             <origin rpy="0.0 0.0 0.0" xyz="${x} ${y} -0.01"/>
-            <parent link="base"/>
+            <parent link="base_link"/>
             <child link="${prefix}_holder"/>
         </joint>
@@ -115,5 +115,5 @@
     <joint name="head_joint" type="fixed">
         <origin xyz="0.1275 0.0 -0.004" rpy="0.0 0.0 0.0"/>
-        <parent link="base"/>
+        <parent link="base_link"/>
         <child link="head"/>
     </joint>
@@ -143,5 +143,5 @@
     <joint name="camera_mount_joint" type="fixed">
         <origin xyz="0.085 0.0 0.06" rpy="0.0 0.0 0.0"/>
-        <parent link="base"/>
+        <parent link="base_link"/>
         <child link="camera_mount"/>
     </joint>
@@ -198,5 +198,5 @@
     <joint name="board_joint" type="fixed">
         <origin xyz="-0.0375 0.0 0.0475" rpy="0.0 0.0 0.0"/>
-        <parent link="base"/>
+        <parent link="base_link"/>
         <child link="board"/>
     </joint>

Commit message: Fix JetRacer robot description: mount offsets, degenerate inertia, import corruption
- Correct lidar/camera mount joint offsets in xacro/urdf (were stale from
  earlier board/camera_mount resizes, leaving both sensors embedded inside
  their mounts instead of sitting on top)
- Clear degenerate zero diagonal-inertia override on the chassis body,
  auto-computed from mass + collision geometry instead
- Remove broken duplicate reference entries (top-level jetracer prim and
  the mujoco/physics/physx Physics variant payloads) causing composition
  errors on load
- Clean up duplicated body0/body1 joint relationships left over from
  repeated re-imports into the same stage
- Disconnect the legacy (non-RTX) IsaacReadLidarPointCloud node, which
  crashes PhysX on Play due to a stale prim-type mismatch; RTX lidar
  pipeline already publishes the point cloud correctly on its own

File: jetracer.urdf (robot description, URDF)
Before this commit: robot jetracer, 12 links, 11 joints
Links:
- added link base_inertial, mass 1.166
- link base_link: mass 1.0 -> None
- link board: mass 0.15 -> 0.001; geometry collision box size=0.145 0.10 0.275; visual box size=0.145 0.10 0.275
- link camera: mass 0.01 -> 0.001
- link camera_mount: mass 0.05 -> 0.001; geometry collision box size=0.01 0.01 0.25; visual box size=0.01 0.01 0.25
- link front_left_wheel: mass 0.05 -> 0.07
- link front_right_wheel: mass 0.05 -> 0.07
- link lidar: mass 0.04 -> 0.001
- link rear_left_wheel: mass 0.05 -> 0.07
- link rear_right_wheel: mass 0.05 -> 0.07
Joints:
- added joint base_inertial_joint: type fixed, parent base_link, child base_inertial, origin xyz=0 0 0 rpy=0 0 0
- joint board_joint: origin xyz=-0.0375 0.0 0.0475 rpy=0.0 0.0 0.0 -> xyz=-0.0375 0.0 0.14614899660969316 rpy=0.0 0.0 0.0
- joint camera_joint: origin xyz=0 0 0.103 rpy=0 0 0 -> xyz=0 0 0.06 rpy=0 1.5708 0
- joint camera_mount_joint: origin xyz=0.085 0.0 0.06 rpy=0.0 0.0 0.0 -> xyz=0.085 0.0 0.10233622380397495 rpy=0.0 0.0 0.0
- joint lidar_joint: origin xyz=0.0 0.0 0.075 rpy=0.0 0.0 0.0 -> xyz=0.0 0.0 0.1575 rpy=0.0 0.0 0.0

File: jetracer.xacro (robot description, xacro)
@@ -21,7 +21,18 @@
             </geometry>
         </collision>
-        <inertial>
-            <mass value="1.0"/>
-            <inertia ixx="0.004067" iyy="0.005042" izz="0.001042" ixy="0" ixz="0" iyz="0"/>
+    </link>
+    <!-- Massless base_link (root) with inertia moved onto this coincident child:
+         KDL/robot_state_publisher doesn't support the tree's root link carrying
+         an inertia. base_link itself must stay the root untouched, since Isaac
+         Sim's odometry bridge externally publishes odom->base_link directly. -->
+    <joint name="base_inertial_joint" type="fixed">
+        <origin rpy="0 0 0" xyz="0 0 0"/>
+        <parent link="base_link"/>
+        <child link="base_inertial"/>
+    </joint>
+    <link name="base_inertial">
+        <inertial>
+            <mass value="1.166"/>
+            <inertia ixx="0.004742" iyy="0.005879" izz="0.001215" ixy="0" ixz="0" iyz="0"/>
         </inertial>
     </link>
@@ -36,6 +47,6 @@
         <link name="${prefix}_wheel">
             <inertial>
-                <mass value="0.05"/>
-                <inertia ixx="0.00000875" iyy="0.00000875" izz="0.0000156" ixy="0" ixz="0" iyz="0"/>
+                <mass value="0.07"/>
+                <inertia ixx="0.00001225" iyy="0.00001225" izz="0.00002184" ixy="0" ixz="0" iyz="0"/>
             </inertial>
             <visual>
@@ -70,6 +81,6 @@
         <link name="${prefix}_wheel">
             <inertial>
-                <mass value="0.05"/>
-                <inertia ixx="0.00000875" iyy="0.00000875" izz="0.0000156" ixy="0" ixz="0" iyz="0"/>
+                <mass value="0.07"/>
+                <inertia ixx="0.00001225" iyy="0.00001225" izz="0.00002184" ixy="0" ixz="0" iyz="0"/>
             </inertial>
             <visual>
@@ -142,5 +153,5 @@
     <!-- Camera -->
     <joint name="camera_mount_joint" type="fixed">
-        <origin xyz="0.085 0.0 0.06" rpy="0.0 0.0 0.0"/>
+        <origin xyz="0.085 0.0 0.10233622380397495" rpy="0.0 0.0 0.0"/>
         <parent link="base_link"/>
         <child link="camera_mount"/>
@@ -149,11 +160,11 @@
         <inertial>
             <origin xyz="0.0 0.0 0.0" rpy="0.0 0.0 0.0"/>
-            <mass value="0.05"/>
-            <inertia ixx="0.0000084" iyy="0.00000017" izz="0.0000084" ixy="0" ixz="0" iyz="0"/>
-        </inertial>
-        <visual>
-            <origin xyz="0.0 0.0 0.0" rpy="0.0 0.0 0.0"/>
-            <geometry>
-                <box size="0.01 0.01 0.20"/>
+            <mass value="0.001"/>
+            <inertia ixx="0.0000001" iyy="0.0000001" izz="0.0000001" ixy="0" ixz="0" iyz="0"/>
+        </inertial>
+        <visual>
+            <origin xyz="0.0 0.0 0.0" rpy="0.0 0.0 0.0"/>
+            <geometry>
+                <box size="0.01 0.01 0.25"/>
             </geometry>
             <material name="mount_red">
@@ -164,10 +175,10 @@
             <origin xyz="0.0 0.0 0.0" rpy="0.0 0.0 0.0"/>
             <geometry>
-                <box size="0.01 0.01 0.20"/>
+                <box size="0.01 0.01 0.25"/>
             </geometry>
         </collision>
     </link>
     <joint name="camera_joint" type="fixed">
-        <origin xyz="0 0 0.103" rpy="0 0 0"/>
+        <origin xyz="0 0 0.06" rpy="0 1.5708 0"/>
         <parent link="camera_mount"/>
         <child link="camera"/>
@@ -176,6 +187,6 @@
         <inertial>
             <origin xyz="0 0 0" rpy="0 0 0"/>
-            <mass value="0.01"/>
-            <inertia ixx="0.00000047" iyy="0.00000047" izz="0.00000028" ixy="0" ixz="0" iyz="0"/>
+            <mass value="0.001"/>
+            <inertia ixx="0.0000001" iyy="0.0000001" izz="0.0000001" ixy="0" ixz="0" iyz="0"/>
         </inertial>
         <visual>
@@ -197,5 +208,5 @@
     <!-- Board -->
     <joint name="board_joint" type="fixed">
-        <origin xyz="-0.0375 0.0 0.0475" rpy="0.0 0.0 0.0"/>
+        <origin xyz="-0.0375 0.0 0.14614899660969316" rpy="0.0 0.0 0.0"/>
         <parent link="base_link"/>
         <child link="board"/>
@@ -205,5 +216,5 @@
             <origin xyz="0 0 0" rpy="0 0 0"/>
             <geometry>
-                <box size="0.145 0.10 0.11"/>
+                <box size="0.145 0.10 0.275"/>
             </geometry>
             <material name="black">
@@ -214,15 +225,15 @@
             <origin xyz="0 0 0" rpy="0 0 0"/>
             <geometry>
-                <box size="0.145 0.10 0.11"/>
-            </geometry>
-        </collision>
-        <inertial>
-            <mass value="0.15"/>
-            <inertia ixx="0.000414" iyy="0.000388" izz="0.000276" ixy="0" ixz="0" iyz="0"/>
+                <box size="0.145 0.10 0.275"/>
+            </geometry>
+        </collision>
+        <inertial>
+            <mass value="0.001"/>
+            <inertia ixx="0.0000001" iyy="0.0000001" izz="0.0000001" ixy="0" ixz="0" iyz="0"/>
         </inertial>
     </link>
     <!-- LiDAR -->
     <joint name="lidar_joint" type="fixed">
-        <origin xyz="0.0 0.0 0.075" rpy="0.0 0.0 0.0"/>
+        <origin xyz="0.0 0.0 0.1575" rpy="0.0 0.0 0.0"/>
         <parent link="board"/>
         <child link="lidar"/>
@@ -231,6 +242,6 @@
         <inertial>
             <origin xyz="0.0 0.0 0.0" rpy="0.0 0.0 0.0"/>
-            <mass value="0.04"/>
-            <inertia ixx="0.0000303" iyy="0.0000303" izz="0.00005" ixy="0" ixz="0" iyz="0"/>
+            <mass value="0.001"/>
+            <inertia ixx="0.0000001" iyy="0.0000001" izz="0.0000001" ixy="0" ixz="0" iyz="0"/>
         </inertial>
         <visual>
